Commit message: 2024-4-19 19：30 训练踏步，但有奇怪的pos_vel超极限问题

File: resources/robots/zq01/urdf/zq_box_foot.urdf (robot description, URDF)
Before this commit: robot zp_humanoid, 13 links, 12 joints
Joints:
- joint JOINT_Y5: limit lower=-0.6 upper=0.6 effort=24 velocity=31 -> lower=-0.6 upper=1.0 effort=24 velocity=31
- joint JOINT_Z5: limit lower=-0.6 upper=0.6 effort=24 velocity=31 -> lower=-0.6 upper=1.0 effort=24 velocity=31

Commit message: 2024-4-19 22：03 发现dof_vel不准问题，用delta_pos计算解决。

File: resources/robots/zq01/urdf/zq_box_foot.urdf (robot description, URDF)
Before this commit: robot zp_humanoid, 13 links, 12 joints
Links:
- link Y1: mass 10 -> 1.528
